File: Electronics/sensoluche_v1_0/sensoluche_v1_0.sch (KiCad schematic (older format))
At the start: 21 parts, among them J1 EXT_IO_AN, J2 TB_2, P1 FSR402_Pressure

Commit message: V1.0 New flex sensors
Parts:
- removed R1, R3, R5, R7, R9: 22K, Resistor_THT:R_Axial_DIN0207_L6.3mm_D2.5mm_P7.62mm_Horizontal, symbol Device:R
- removed R10, R2, R4, R6, R8: 100K, Resistor_THT:R_Axial_DIN0207_L6.3mm_D2.5mm_P7.62mm_Horizontal, symbol Device:R
- added J2: EXT_IO_AN, Connector_PinHeader_2.54mm:PinHeader_2x05_P2.54mm_Vertical, symbol Connector_Generic:Conn_02x05_Top_Bottom
- renumbered J2 to J3, R11 to R1
Connections:
- net +3V3: now also J2.9 (Pin_9)
- net A_Adventure: now also A1.24 (A5), F5.3; no longer A1.25 (A6)
- net A_Comedy: now also A1.20 (A1), F1.3; no longer A1.21 (A2)
- net A_Drama: now also A1.23 (A4), F4.3; no longer A1.24 (A5)
- net A_Horror: now also A1.21 (A2), F2.3; no longer A1.22 (A3)
- net A_Pressure: now also A1.19 (A0), A1.6 (D3); no longer A1.20 (A1)
- net A_Romance: now also A1.22 (A3), F3.3; no longer A1.23 (A4)
- net D_Vibration: now also A1.5 (D2); no longer A1.10 (D7)
- net GND: now also J2.10 (Pin_10)
- net D1_TX: now reaches A1.1 (D1/TX)
- net D1_TX: now also J2.2 (Pin_2)
- net D0_RX: now reaches A1.2 (D0/RX)
- net D0_RX: now also J2.1 (Pin_1)
- net A0 renamed A6
- net A6: now also A1.25 (A6); no longer A1.19 (A0)
- net D_Adventure renamed D6
- net D6: now also J2.5 (Pin_5); no longer F5.3
- removed net D_Comedy: A1.5 (D2), F1.3
- net D_Drama renamed D5
- net D5: now also J2.4 (Pin_4); no longer F4.3
- removed net D_Horror: A1.6 (D3), F2.3
- net D_Romance renamed D4
- net D4: now also J2.3 (Pin_3); no longer F3.3
- new net D7: A1.10 (D7), J2.6 (Pin_6)
Other:
- moved on the sheet: J1, J3
